Commit message: Labs 7-9: Add source code, models, English docs, and tests
- Lab 7 (Locomotion): G1 model, balance controller, LIPM planner, walking demo
- Lab 8 (Whole-Body): QP controller, tasks, contact model, walking+manipulation
- Lab 9 (VLA): Scene setup, demo collector, domain randomizer, vision encoder

https://claude.ai/code/session_01JZV6rU3Rh2wbK1eeETfjbB

File: lab-7-locomotion/models/g1_humanoid.urdf (robot description, URDF)
Before this commit: robot g1_humanoid, 19 links, 18 joints
Links:
- link left_shin: geometry collision cylinder length=0.30 radius=0.045
- link left_thigh: geometry collision cylinder length=0.30 radius=0.05
- link right_shin: geometry collision cylinder length=0.30 radius=0.045
- link right_thigh: geometry collision cylinder length=0.30 radius=0.05
Joints:
- joint root_joint: origin xyz=0 0 0.82 rpy=0 0 0 -> xyz=0 0 0 rpy=0 0 0; type floating -> fixed
