Commit message: Add video production pipeline for MuJoCo Robotics Lab
- Introduced a new module `video_producer.py` that implements a reusable video production pipeline.
- The pipeline standardizes the workflow into three phases: animated metrics presentation, simulation recording, and final video composition.
- Added functionality for creating metrics figures with customizable plots and overlays.
- Implemented a streaming video writer using ffmpeg for efficient video frame writing.
- Included methods for rendering simulation scenes with trace visualization and overlays.
- Created utility functions for generating title and end cards for the final video.
- Added a convenience function `generate_demo_video` to encapsulate the entire video generation process.

File: lab-3-dynamics-force-control/models/ur5e.urdf (robot description, URDF)
Before this commit: robot ur5e, 9 links, 8 joints
Links:
- added link pinch_link, mass 1e-6
- link base_link: mass 2.4429 -> 4.0; geometry collision cylinder length=0.12 radius=0.06
- link ee_link: mass 0.0972 -> 1.0526083388
- link forearm_link: mass 3.0216 -> 2.275; geometry collision cylinder length=0.392 radius=0.038
- link shoulder_link: mass 2.0736 -> 3.7; geometry collision cylinder length=0.12 radius=0.06
- link upper_arm_link: mass 3.7887 -> 8.393; geometry collision cylinder length=0.425 radius=0.05
- link wrist_1_link: mass 0.8128 -> 1.219; geometry collision cylinder length=0.1 radius=0.04
- link wrist_2_link: mass 0.6150 -> 1.219; geometry collision cylinder length=0.1 radius=0.04
- link wrist_3_link: mass 0.5593 -> 0.1889; geometry collision cylinder length=0.04 radius=0.04
Joints:
- added joint pinch_fixed_joint: type fixed, parent ee_link, child pinch_link, origin xyz=0 0 0.1558 rpy=0 0 0
- joint ee_fixed_joint: origin xyz=0 0 0.135 rpy=0 0 0 -> xyz=0 0.1 0 rpy=-1.5707963267948966 0 0
- joint elbow_joint: axis 0 0 1 -> 0 1 0; limit lower=-6.28318530718 upper=6.28318530718 effort=150.0 velocity=3.14 -> lower=-3.14159265359 upper=3.14159265359 effort=150.0 velocity=3.14; origin xyz=-0.425 0 0 rpy=0 0 0 -> xyz=0 -0.131 0.425 rpy=0 0 0
- joint shoulder_lift_joint: axis 0 0 1 -> 0 1 0; origin xyz=0 0 0 rpy=1.5707963267948966 0 0 -> xyz=0 0.138 0 rpy=0 1.5707963267948966 0
- joint shoulder_pan_joint: origin xyz=0 0 0.1625 rpy=0 0 0 -> xyz=0 0 0.163 rpy=0 0 0
- joint world_joint: origin xyz=0 0 0 rpy=0 0 0 -> xyz=0 0 0 rpy=0 0 3.14159265358979
- joint wrist_1_joint: axis 0 0 1 -> 0 1 0; origin xyz=-0.3922 0 0.1333 rpy=0 0 0 -> xyz=0 0 0.392 rpy=0 1.5707963267948966 0
- joint wrist_2_joint: origin xyz=0 0 0.0997 rpy=1.5707963267948966 0 0 -> xyz=0 0.127 0 rpy=0 0 0
- joint wrist_3_joint: axis 0 0 1 -> 0 1 0; origin xyz=0 0 0.0996 rpy=-1.5707963267948966 0 0 -> xyz=0 0 0.1 rpy=0 0 0
